File: hardware/PiPicoCNCShield/DriverCarrier.kicad_sch (KiCad schematic)
At the start: 5 parts

Commit message: Initial PCB design
Initial PCB design
Parts:
- J25: renamed from J?; footprint (none) -> Connector_PinHeader_2.54mm:PinHeader_1x03_P2.54mm_Vertical
- J27: renamed from J?; footprint (none) -> Connector_JST:JST_XH_B4B-XH-A_1x04_P2.50mm_Vertical
- J28: renamed from J?; footprint (none) -> Connector_JST:JST_XH_B3B-XH-A_1x03_P2.50mm_Vertical
- U5: renamed from U?; footprint (none) -> DriverCarrier:DriverCarrier
- gave numbers to parts that had none: 1
Changed lines of the file:
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@@
   (symbol (lib_id "Connector_Generic:Conn_02x03_Odd_Even") (at 81.28 75.565 270)
     (in_bom yes) (on_board yes) (fields_autoplaced)
-    (property "Reference" "J?" (id 0) (at 86.36 75.5649 90)
+    (property "Reference" "J26" (id 0) (at 86.36 75.5649 90)
       (effects (font (size 1.27 1.27)) (justify left))
     )
@@
   (symbol (lib_id "Connector_Generic:Conn_01x04") (at 160.02 84.455 0)
     (in_bom yes) (on_board yes) (fields_autoplaced)
-    (property "Reference" "J?" (id 0) (at 162.56 84.4549 0)
+    (property "Reference" "J27" (id 0) (at 162.56 84.4549 0)
       (effects (font (size 1.27 1.27)) (justify left))
     )
@@
       (effects (font (size 1.27 1.27)) (justify left))
     )
-    (property "Footprint" "" (id 2) (at 160.02 84.455 0)
+    (property "Footprint" "Connector_JST:JST_XH_B4B-XH-A_1x04_P2.50mm_Vertical" (id 2) (at 160.02 84.455 0)
       (effects (font (size 1.27 1.27)) hide)
     )
@@
   (symbol (lib_id "Connector_Generic:Conn_01x03") (at 157.48 112.395 180)
     (in_bom yes) (on_board yes)
-    (property "Reference" "J?" (id 0) (at 157.48 102.87 0))
+    (property "Reference" "J28" (id 0) (at 157.48 102.87 0))
     (property "Value" "D_EndStop" (id 1) (at 157.48 105.41 0))
-    (property "Footprint" "" (id 2) (at 157.48 112.395 0)
+    (property "Footprint" "Connector_JST:JST_XH_B3B-XH-A_1x03_P2.50mm_Vertical" (id 2) (at 157.48 112.395 0)
       (effects (font (size 1.27 1.27)) hide)
     )
@@
   (symbol (lib_id "Drivers:DriverCarrier") (at 127 90.805 0)
     (in_bom yes) (on_board yes) (fields_autoplaced)
-    (property "Reference" "U?" (id 0) (at 126.365 67.31 0))
+    (property "Reference" "U5" (id 0) (at 126.365 67.31 0))
     (property "Value" "DriverCarrier" (id 1) (at 126.365 69.85 0))
-    (property "Footprint" "" (id 2) (at 127 90.805 0)
+    (property "Footprint" "DriverCarrier:DriverCarrier" (id 2) (at 127 90.805 0)
       (effects (font (size 1.27 1.27)) hide)
     )
@@
   (symbol (lib_id "Connector_Generic:Conn_01x03") (at 189.865 74.295 0)
     (in_bom yes) (on_board yes) (fields_autoplaced)
-    (property "Reference" "J?" (id 0) (at 193.04 73.0249 0)
+    (property "Reference" "J25" (id 0) (at 193.04 73.0249 0)
       (effects (font (size 1.27 1.27)) (justify left))
     )
@@
       (effects (font (size 1.27 1.27)) (justify left))
     )
-    (property "Footprint" "" (id 2) (at 189.865 74.295 0)
+    (property "Footprint" "Connector_PinHeader_2.54mm:PinHeader_1x03_P2.54mm_Vertical" (id 2) (at 189.865 74.295 0)
       (effects (font (size 1.27 1.27)) hide)
     )
