File: hardware/PiPicoCNCShield/PiPicoCNCShield.kicad_pcb (KiCad board)
At the start: 2 copper layers, 100 x 100 mm, 41 parts, among them J1 I2C_Conn, J10 IO_6, J11 IO_3, J12 IO_9, J13 D_MotorVoltageJumper, J14 D_MicrostepJumper, J15 D_MOTOR_Conn, J16 D_EndStop, J17 D_MotorVoltageJumper, J18 D_MicrostepJumper, J19 D_MOTOR_Conn, J2 I2C_Conn, J20 D_EndStop, J21 D_MotorVoltageJumper, J22 D_MicrostepJumper, J23 D_MOTOR_Conn, J24 D_EndStop, J25 D_MotorVoltageJumper, J26 D_MicrostepJumper, J27 D_MOTOR_Conn, J28 D_EndStop, J29 POWER_CONN, J3 I2C_Conn, J30 UART, J4 IO_1, J5 IO_4, J6 IO_7, J7 IO_2, J8 IO_5, J9 IO_8, U1 Pico, U2 DriverCarrier, U3 DriverCarrier, U4 DriverCarrier, U5 DriverCarrier

Commit message: Test run
Parts:
- R1: footprint Resistor_SMD:R_0603_1608Metric_Pad0.98x0.95mm_HandSolder -> Resistor_SMD:R_0805_2012Metric_Pad1.20x1.40mm_HandSolder
- moved R1 6.27 mm to (193.0, 65.8)
- moved D1 4.85 mm to (193.0, 59.8)
Routing:
- net GND: track 42.1 -> 48.6 mm
- net Net-(D1-Pad2): track 4.27 -> 6.24 mm
- net LED: track 10.1 -> 11.8 mm
- net D1_STEP: track 31.8 -> 30.3 mm
Other:
- board text added: "2 1"
- board text added: "3v3"
- board text added: "Endstop"
- board text added: "H L"
- board text added: "MOTOR 1"
- board text added: "MOTOR 2"
- board text added: "MOTOR 3"
- board text added: "MOTOR 4"
- board text added: "VM1"
- board text added: "VM2"
