File: hardware/PiPicoCNCShield/PiPicoCNCShield.kicad_sch (KiCad schematic)
At the start: 30 parts, among them J1 D1_MicrostepJumper, U1 Pico, U2 DriverCarrier1

Commit message: Driver Carrier sub-schematic
Driver Carrier sub-schematic
Parts:
- removed J1: D1_MicrostepJumper, Connector_PinHeader_2.54mm:PinHeader_2x03_P2.54mm_Vertical, symbol Connector_Generic:Conn_02x03_Odd_Even
- removed J?: D1_MotorVoltageJumper, symbol Connector_Generic:Conn_01x03
- removed J?: D3_MOTOR_Conn, symbol Connector_Generic:Conn_01x04
- removed J?: D2_MicrostepJumper, Connector_PinHeader_2.54mm:PinHeader_2x03_P2.54mm_Vertical, symbol Connector_Generic:Conn_02x03_Odd_Even
- removed J?: D3_EndStop, symbol Connector_Generic:Conn_01x03
- removed J?: D3_MicrostepJumper, Connector_PinHeader_2.54mm:PinHeader_2x03_P2.54mm_Vertical, symbol Connector_Generic:Conn_02x03_Odd_Even
- removed J?: D2_EndStop, symbol Connector_Generic:Conn_01x03
- removed J?: D2_MotorVoltageJumper, symbol Connector_Generic:Conn_01x03
- removed J?: D1_EndStop, symbol Connector_Generic:Conn_01x03
- removed J?: D2_MOTOR_Conn, symbol Connector_Generic:Conn_01x04
- removed J?: D3_MotorVoltageJumper, symbol Connector_Generic:Conn_01x03
- removed J?: D1_MOTOR_Conn, symbol Connector_Generic:Conn_01x04
- removed U2: DriverCarrier1, symbol Drivers:DriverCarrier
- removed U?: DriverCarrier2, symbol Drivers:DriverCarrier
- removed U?: DriverCarrier3, symbol Drivers:DriverCarrier
Connections:
- net IO_6_Sig renamed IO_6_Sig_D4_EN
- net IO_7_Sig renamed IO_7_Sig_D4_STEP
- net IO_8_Sig renamed IO_8_Sig_D4_DIR
- net IO_9_Sig renamed IO_9_Sig_D4_ENDSTOP
Other:
- added sheet DriverCarrier1 (DriverCarrier.kicad_sch)
- added sheet DriverCarrier2 (DriverCarrier.kicad_sch)
- added sheet DriverCarrier3 (DriverCarrier.kicad_sch)
- added sheet DriverCarrier4 (DriverCarrier.kicad_sch)
- moved on the sheet: J?

Commit message: Initial PCB design
Initial PCB design
Parts:
- added H1, H2, H3, H4: MountingHole_Pad, MountingHole:MountingHole_3.2mm_M3_ISO7380_Pad, symbol Mechanical:MountingHole_Pad
- added J29: POWER_CONN, Connector_Phoenix_MC_HighVoltage:PhoenixContact_MC_1,5_6-G-5.08_1x06_P5.08mm_Horizontal, symbol Connector_Generic:Conn_01x06
- added J30: UART, Connector_JST:JST_XH_B3B-XH-A_1x03_P2.50mm_Vertical, symbol Connector_Generic:Conn_01x03
- J1, J2, J3: renamed from J?; footprint (none) -> Connector_JST:JST_XH_B4B-XH-A_1x04_P2.50mm_Vertical
- J10, J11, J12, J4, J5, J6, J7, J8, J9: renamed from J?; footprint (none) -> Connector_JST:JST_XH_B3B-XH-A_1x03_P2.50mm_Vertical
- U1: footprint RPi_Pico:RPi_Pico_SMD_TH -> MCU_RaspberryPi_and_Boards:RPi_Pico_SMD_TH
- gave numbers to parts that had none: 2
Connections:
- net +12V: now also J29.4 (Pin_4)
- net +3V3: now also J29.2 (Pin_2)
- net D1_DIR: now also U1.4 (GPIO2); no longer U1.6 (GPIO4)
- net D1_EN: now also U1.6 (GPIO4); no longer U1.4 (GPIO2)
- net D2_DIR: now also U1.9 (GPIO6); no longer U1.11 (GPIO8)
- net D2_EN: now also U1.11 (GPIO8); no longer U1.9 (GPIO6)
- net D3_DIR: now also U1.14 (GPIO10); no longer U1.16 (GPIO12)
- net D3_EN: now also U1.16 (GPIO12); no longer U1.14 (GPIO10)
- net GND: now also H1.1, H2.1, H3.1, H4.1, J29.1 (Pin_1), J29.3 (Pin_3), J29.5 (Pin_5), J30.1 (Pin_1)
- net RX: now also J30.2 (Pin_2)
- net TX: now also J30.3 (Pin_3)
- net VAA: now also J29.6 (Pin_6)
- net +5V: no longer names the net of U1.40 (VBUS)
- net IO_7_Sig_D4_STEP renamed IO_7_Sig_D4_ENDSTOP
- net IO_8_Sig_D4_DIR renamed IO_8_Sig_D4_STEP
- net IO_9_Sig_D4_ENDSTOP renamed IO_9_Sig_D4_DIR
Other:
- sheet DriverCarrier1 renamed #DriverCarrier1

Commit message: Test run
Parts:
- R1: footprint Resistor_SMD:R_0603_1608Metric_Pad0.98x0.95mm_HandSolder -> Resistor_SMD:R_0805_2012Metric_Pad1.20x1.40mm_HandSolder
Changed lines of the file:
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@@
     (property "Reference" "R1" (id 0) (at 144.145 149.86 90))
     (property "Value" "R" (id 1) (at 144.145 152.4 90))
-    (property "Footprint" "Resistor_SMD:R_0603_1608Metric_Pad0.98x0.95mm_HandSolder" (id 2) (at 144.145 157.988 90)
+    (property "Footprint" "Resistor_SMD:R_0805_2012Metric_Pad1.20x1.40mm_HandSolder" (id 2) (at 144.145 157.988 90)
       (effects (font (size 1.27 1.27)) hide)
     )
@@
     )
     (path "/aa9a7955-6f79-4ab6-956c-0ea64130df2f"
-      (reference "R1") (unit 1) (value "R") (footprint "Resistor_SMD:R_0603_1608Metric_Pad0.98x0.95mm_HandSolder")
+      (reference "R1") (unit 1) (value "R") (footprint "Resistor_SMD:R_0805_2012Metric_Pad1.20x1.40mm_HandSolder")
     )
     (path "/03817d20-266c-4a32-a072-56f20d48d854"
